File: PCB/KCVGA 1.1.brd (EAGLE design)
At the start: 50 x 50 mm, 64 parts, among them IC1 XC3S50ATQ144, IC2 PIC32MX250F128, IC3 M68AW128MND, IC4 AP1117-1.2, IC5 AP1117-3.3, IC6 74245ADB, X1 D-SUB15, X3 MINI-USB

Commit message: PCB v1.1 production release
Routing:
- net !FPGA_RESET: track 16.1 -> 22.9 mm
Changed lines of the file:
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@@
 <grid distance="12.5" unitdist="mil" unit="mil" style="lines" multiple="1" display="yes" altdistance="6.25" altunitdist="mil" altunit="mil"/>
 <layers>
-<layer number="1" name="Top" color="4" fill="1" visible="no" active="yes"/>
-<layer number="16" name="Bottom" color="1" fill="1" visible="no" active="yes"/>
-<layer number="17" name="Pads" color="2" fill="1" visible="no" active="yes"/>
-<layer number="18" name="Vias" color="2" fill="1" visible="no" active="yes"/>
+<layer number="1" name="Top" color="4" fill="1" visible="yes" active="yes"/>
+<layer number="16" name="Bottom" color="1" fill="1" visible="yes" active="yes"/>
+<layer number="17" name="Pads" color="2" fill="1" visible="yes" active="yes"/>
+<layer number="18" name="Vias" color="2" fill="1" visible="yes" active="yes"/>
 <layer number="19" name="Unrouted" color="6" fill="1" visible="yes" active="yes"/>
 <layer number="20" name="Dimension" color="15" fill="1" visible="yes" active="yes"/>
 <layer number="21" name="tPlace" color="7" fill="1" visible="yes" active="yes"/>
-<layer number="22" name="bPlace" color="7" fill="1" visible="no" active="yes"/>
-<layer number="23" name="tOrigins" color="15" fill="1" visible="no" active="yes"/>
-<layer number="24" name="bOrigins" color="15" fill="1" visible="no" active="yes"/>
+<layer number="22" name="bPlace" color="7" fill="1" visible="yes" active="yes"/>
+<layer number="23" name="tOrigins" color="15" fill="1" visible="yes" active="yes"/>
+<layer number="24" name="bOrigins" color="15" fill="1" visible="yes" active="yes"/>
 <layer number="25" name="tNames" color="7" fill="1" visible="yes" active="yes"/>
 <layer number="26" name="bNames" color="7" fill="1" visible="no" active="yes"/>
 <layer number="27" name="tValues" color="7" fill="1" visible="no" active="yes"/>
 <layer number="28" name="bValues" color="7" fill="1" visible="no" active="yes"/>
-<layer number="29" name="tStop" color="7" fill="3" visible="yes" active="yes"/>
+<layer number="29" name="tStop" color="7" fill="3" visible="no" active="yes"/>
 <layer number="30" name="bStop" color="7" fill="6" visible="no" active="yes"/>
 <layer number="31" name="tCream" color="7" fill="4" visible="no" active="yes"/>
@@
 <layer number="39" name="tKeepout" color="4" fill="11" visible="no" active="yes"/>
 <layer number="40" name="bKeepout" color="1" fill="11" visible="no" active="yes"/>
-<layer number="41" name="tRestrict" color="4" fill="10" visible="yes" active="yes"/>
+<layer number="41" name="tRestrict" color="4" fill="10" visible="no" active="yes"/>
 <layer number="42" name="bRestrict" color="1" fill="10" visible="yes" active="yes"/>
 <layer number="43" name="vRestrict" color="2" fill="10" visible="yes" active="yes"/>
@@
 <wire x1="18.3007" y1="32.0675" x2="18.161" y2="32.2072" width="0.1524" layer="1"/>
 <wire x1="17.145" y1="30.24" x2="17.2225" y2="30.1625" width="0.1524" layer="1"/>
-<wire x1="35.1065" y1="4.7625" x2="34.925" y2="4.7625" width="0.1524" layer="1"/>
 <wire x1="32.5" y1="16.84" x2="32.5" y2="18.6175" width="0.1524" layer="1"/>
 <wire x1="32.5" y1="18.6175" x2="32.385" y2="18.7325" width="0.1524" layer="1"/>
@@
 <via x="29.845" y="30.48" extent="1-16" drill="0.381"/>
 <via x="43.18" y="46.99" extent="1-16" drill="0.381"/>
-<via x="18.415" y="23.8125" extent="1-16" drill="0.381"/>
+<via x="18.415" y="23.495" extent="1-16" drill="0.381"/>
 <via x="23.8125" y="22.5425" extent="1-16" drill="0.381"/>
 <via x="25.0825" y="19.3675" extent="1-16" drill="0.381"/>
@@
 <contactref element="IC2" pad="17"/>
 <contactref element="IC1" pad="P28"/>
-<wire x1="20.65" y1="23.19" x2="19.38" y2="23.19" width="0.1524" layer="1"/>
-<wire x1="19.38" y1="23.19" x2="18.7325" y2="22.5425" width="0.1524" layer="1"/>
-<wire x1="18.7325" y1="22.5425" x2="18.0975" y2="22.5425" width="0.1524" layer="1"/>
+<wire x1="20.65" y1="23.19" x2="19.6975" y2="23.19" width="0.1524" layer="1"/>
+<wire x1="19.6975" y1="23.19" x2="19.05" y2="22.5425" width="0.1524" layer="1"/>
+<wire x1="19.05" y1="22.5425" x2="18.0975" y2="22.5425" width="0.1524" layer="1"/>
 <wire x1="18.0975" y1="22.5425" x2="17.3949875" y2="21.8399875" width="0.1524" layer="1"/>
 <wire x1="14.729890625" y1="21.8399875" x2="17.3949875" y2="21.8399875" width="0.1524" layer="1"/>
@@
 <wire x1="14.729890625" y1="22.489996875" x2="17.409996875" y2="22.489996875" width="0.1524" layer="1"/>
 <wire x1="17.409996875" y1="22.489996875" x2="17.78" y2="22.86" width="0.1524" layer="1"/>
-<wire x1="17.78" y1="22.86" x2="18.415" y2="22.86" width="0.1524" layer="1"/>
-<wire x1="18.415" y1="22.86" x2="19.245" y2="23.69" width="0.1524" layer="1"/>
-<wire x1="20.65" y1="23.69" x2="19.245" y2="23.69" width="0.1524" layer="1"/>
+<wire x1="17.78" y1="22.86" x2="18.7325" y2="22.86" width="0.1524" layer="1"/>
+<wire x1="18.7325" y1="22.86" x2="19.5625" y2="23.69" width="0.1524" layer="1"/>
+<wire x1="20.65" y1="23.69" x2="19.5625" y2="23.69" width="0.1524" layer="1"/>
 </signal>
 <signal name="N$10">
@@
 <wire x1="19.7525" y1="27.69" x2="19.05" y2="26.9875" width="0.1524" layer="1"/>
 <via x="19.05" y="26.9875" extent="1-16" drill="0.381"/>
-<wire x1="19.05" y1="26.9875" x2="18.415" y2="27.6225" width="0.1524" layer="16"/>
-<wire x1="18.415" y1="27.6225" x2="12.7" y2="27.6225" width="0.1524" layer="16"/>
+<wire x1="17.145" y1="27.6225" x2="12.7" y2="27.6225" width="0.1524" layer="16"/>
 <wire x1="12.7" y1="27.6225" x2="12.3825" y2="27.305" width="0.1524" layer="16"/>
 <wire x1="12.3825" y1="27.305" x2="11.7475" y2="27.305" width="0.1524" layer="16"/>
@@
 <wire x1="8.5725" y1="23.1775" x2="7.5326" y2="23.1775" width="0.1524" layer="1"/>
 <wire x1="7.5326" y1="23.1775" x2="7.495109375" y2="23.140009375" width="0.1524" layer="1"/>
+<wire x1="17.145" y1="27.6225" x2="17.145" y2="24.13" width="0.1524" layer="16"/>
+<wire x1="17.145" y1="24.13" x2="19.3675" y2="24.13" width="0.1524" layer="16"/>
+<wire x1="19.3675" y1="24.13" x2="19.685" y2="24.4475" width="0.1524" layer="16"/>
+<wire x1="19.685" y1="24.4475" x2="19.685" y2="26.3525" width="0.1524" layer="16"/>
+<wire x1="19.685" y1="26.3525" x2="19.05" y2="26.9875" width="0.1524" layer="16"/>
 </signal>
 <signal name="JP5">
